File: Media/pcb/PCB.brd (EAGLE design)
At the start: 78.7 x 194 mm, 152 parts, among them IC3 MLX90393ELW-ABA-011-SP, IC5 STM32F407VGT6, Q11 8Mhz

Commit message: fixed layout and schematics
Parts:
- moved R50 0.51 mm to (28.2, 71.1), turned to 180 degrees
Connections:
- net ESP_GPIO2: now also R50.2; no longer R50.1
- net GND: now also R50.1
- net VCC: no longer R50.2
Routing:
- net VCC: track 567.0 -> 563.8 mm, vias 35 -> 33
Changed lines of the file:
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@@
 <attribute name="VALUE" x="42.545" y="105.41" size="1.27" layer="28" rot="MR0"/>
 </element>
-<element name="R50" library="rcl" library_urn="urn:adsk.eagle:library:334" package="R0805" package3d_urn="urn:adsk.eagle:package:23553/2" value="100K" x="27.686" y="71.12">
-<attribute name="NAME" x="27.051" y="72.39" size="1.27" layer="25"/>
-<attribute name="SPICEPREFIX" value="R" x="27.686" y="71.12" size="1.778" layer="27" display="off"/>
-<attribute name="VALUE" x="27.051" y="68.58" size="1.27" layer="27"/>
+<element name="R50" library="rcl" library_urn="urn:adsk.eagle:library:334" package="R0805" package3d_urn="urn:adsk.eagle:package:23553/2" value="100K" x="28.194" y="71.12" rot="R180">
+<attribute name="NAME" x="28.829" y="69.85" size="1.27" layer="25" rot="R180"/>
+<attribute name="SPICEPREFIX" value="R" x="28.194" y="71.12" size="1.778" layer="27" rot="R180" display="off"/>
+<attribute name="VALUE" x="28.829" y="73.66" size="1.27" layer="27" rot="R180"/>
 </element>
 <element name="R51" library="rcl" library_urn="urn:adsk.eagle:library:334" package="R0805" package3d_urn="urn:adsk.eagle:package:23553/2" value="510" x="27.686" y="55.88">
@@
 <contactref element="R53" pad="1"/>
 <wire x1="49.53" y1="124.308" x2="49.682" y2="124.46" width="0.254" layer="16"/>
+<contactref element="R50" pad="1"/>
 <wire x1="71.12" y1="30.48" x2="73.66" y2="40.64" width="0" layer="19" extent="1-1"/>
 <wire x1="70.358" y1="145.288" x2="68.58" y2="129.54" width="0" layer="19" extent="1-1"/>
@@
 <contactref element="R49" pad="2"/>
 <contactref element="R36" pad="2"/>
-<contactref element="R50" pad="2"/>
 <contactref element="R52" pad="1"/>
 <contactref element="R55" pad="2"/>
@@
 <wire x1="22.606" y1="115.509" x2="26.67" y2="115.509" width="0.254" layer="1"/>
 <wire x1="26.67" y1="115.509" x2="26.736" y2="115.443" width="0.254" layer="1"/>
-<via x="28.636" y="71.12" extent="1-16" drill="0.35"/>
-<wire x1="28.636" y1="71.12" x2="31.75" y2="71.12" width="0.254" layer="16"/>
-<via x="31.75" y="71.12" extent="1-16" drill="0.35"/>
 <via x="36.449" y="74.737" extent="1-16" drill="0.35"/>
 <wire x1="36.449" y1="74.737" x2="31.811" y2="74.737" width="0.254" layer="16"/>
@@
 <contactref element="ESP8266_HEADER" pad="3"/>
 <contactref element="ESP_DEBUG" pad="7"/>
-<contactref element="R50" pad="1"/>
 <wire x1="11.43" y1="52.07" x2="11.43" y2="66.04" width="0.254" layer="1"/>
 <via x="11.43" y="66.04" extent="1-16" drill="0.35"/>
@@
 <wire x1="19.05" y1="40.64" x2="17.1958" y2="38.7858" width="0.254" layer="1"/>
 <wire x1="17.1958" y1="38.7858" x2="13.51759375" y2="38.7858" width="0.254" layer="1"/>
-<wire x1="26.736" y1="71.12" x2="26.67" y2="71.054" width="0.254" layer="1"/>
-<wire x1="26.67" y1="71.054" x2="26.67" y2="66.04" width="0.254" layer="1"/>
+<contactref element="R50" pad="2"/>
+<wire x1="26.67" y1="66.04" x2="26.67" y2="70.546" width="0.254" layer="1"/>
+<wire x1="26.67" y1="70.546" x2="27.244" y2="71.12" width="0.254" layer="1"/>
 </signal>
 <signal name="N$67">
