File: Media/pcb/PCB.sch (EAGLE design)
At the start: 152 parts, among them IC3 MLX90393ELW-ABA-011-SP, IC5 STM32F407VGT6, Q11 8Mhz

Commit message: fixed layout and schematics
Connections:
- net ESP_GPIO2: now also R50.2; no longer R50.1
- net GND: now also R50.1
- net VCC: no longer R50.2
Other:
- moved on the sheet: R50
Changed lines of the file:
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@@
 <attribute name="VALUE" x="120.65" y="17.018" size="1.778" layer="96"/>
 </instance>
-<instance part="R50" gate="G$1" x="-7.62" y="40.64" rot="R90">
-<attribute name="NAME" x="-9.1186" y="36.83" size="1.778" layer="95" rot="R90"/>
-<attribute name="VALUE" x="-4.318" y="36.83" size="1.778" layer="96" rot="R90"/>
+<instance part="R50" gate="G$1" x="-7.62" y="17.78" rot="R90">
+<attribute name="NAME" x="-9.1186" y="13.97" size="1.778" layer="95" rot="R90"/>
+<attribute name="VALUE" x="-4.318" y="13.97" size="1.778" layer="96" rot="R90"/>
 </instance>
 <instance part="R51" gate="G$1" x="0" y="17.78" rot="R270">
@@
 <wire x1="0" y1="12.7" x2="0" y2="7.62" width="0.1524" layer="91"/>
 <label x="0" y="7.62" size="1.778" layer="95" rot="R90"/>
+<pinref part="R50" gate="G$1" pin="1"/>
+<wire x1="-7.62" y1="12.7" x2="0" y2="12.7" width="0.1524" layer="91"/>
+<junction x="0" y="12.7"/>
 </segment>
 <segment>
@@
 <wire x1="-7.62" y1="48.26" x2="0" y2="48.26" width="0.1524" layer="91"/>
 <pinref part="R36" gate="G$1" pin="2"/>
-<pinref part="R50" gate="G$1" pin="2"/>
-<wire x1="-7.62" y1="48.26" x2="-7.62" y2="45.72" width="0.1524" layer="91"/>
 </segment>
 <segment>
@@
 <wire x1="-5.08" y1="25.4" x2="-7.62" y2="25.4" width="0.1524" layer="91"/>
 <label x="-17.78" y="25.4" size="1.778" layer="95"/>
-<pinref part="R50" gate="G$1" pin="1"/>
 <wire x1="-7.62" y1="25.4" x2="-17.78" y2="25.4" width="0.1524" layer="91"/>
-<wire x1="-7.62" y1="35.56" x2="-7.62" y2="25.4" width="0.1524" layer="91"/>
+<pinref part="R50" gate="G$1" pin="2"/>
+<wire x1="-7.62" y1="25.4" x2="-7.62" y2="22.86" width="0.1524" layer="91"/>
 <junction x="-7.62" y="25.4"/>
 </segment>
